File: SRC/USB_C_HUB/Variable Voltage Source.sch (KiCad schematic (older format))
At the start: 28 parts

Commit message: With ST PD controller(sink)100W
Parts:
- removed C?: 1nF, symbol Device:C
- removed C?: 0.1uF, symbol Device:C
- removed C? (x2): 22uF, symbol Device:C
- removed C? (x2): 100pF, symbol Device:C
- removed D? (x3): SMAJ30A, Diode_SMD:D_SMB, symbol Diode:SM6T30A
- removed D?: PDS1040, Diode_SMD:D_PowerDI-5, symbol Diode:SB140
- removed L?: 10uH, symbol OLIMEX_RCL:INDUCTOR_SMALL
- removed Q? (x3): BSH105,215, Package_TO_SOT_SMD:SC-59, symbol dk_Transistors-FETs-MOSFETs-Single:2N7002P_215
- removed R?: 270, symbol Device:R_US
- removed R?: 47.5K, symbol Device:R_US
- removed R? (x4): 100K, symbol Device:R_US
- removed R?: 11K, symbol Device:R_US
- removed R?: 30K, symbol Device:R_US
- removed R?: 9.53K, symbol Device:R_US
- removed R?: 8.87K_603, symbol Device:R_US
- removed R?: 3.65K_603, symbol Device:R_US
- removed R?: 2.2K_805, symbol Device:R_US
- removed U?: LM3489QMM, symbol usb_hub:LM3489QMM
- removed U?: CWDM3011P, symbol usb_hub:CWDM3011P
Connections:
- net labels removed: GND, POWER_LVL1, POWER_LVL2, POWER_LVL3, SYS_PWR
- wire segments 97 -> 0
Other:
- note removed: "FEEDBACK PATH\n(USED TO SET THE DESIRED VOLTAGE)"
