File: SRC/USB_C_HUB/ST_PD CHARGING CONTROLLER.sch (KiCad schematic (older format))
At the start: 15 parts

Commit message: With ST PD controller(sink)100W
Parts:
- added D?: ESDA25P35, digikey-footprints:SOD-523, symbol dk_TVS-Diodes:ESD5Z3_3T1G
Connections:
- net GND: now also D?.A, D?.A
- net PWR_IN: now also D?.K
- net at R?.2, U?.9 (DISCH): no longer D?.A
Changed lines of the file:
@@
 $Descr A4 11693 8268
 encoding utf-8
-Sheet 2 3
+Sheet 3 4
 Title ""
 Date ""
@@
 Wire Wire Line
 	2375 2175 2375 1575
-Wire Wire Line
-	2375 1575 2300 1575
 Wire Wire Line
 	2375 1575 2800 1575
@@
 Wire Wire Line
 	4925 3075 6800 3075
-Connection ~ 6800 3075
-Wire Wire Line
-	6800 3075 7150 3075
 Text Label 3450 2475 2    39   ~ 0
 CC1_PWR
@@
 NoConn ~ 3725 2275
 NoConn ~ 3725 3475
-Text HLabel 2300 1575 0    50   Input ~ 0
+Text HLabel 1375 1575 0    50   Input ~ 0
 PWR_IN
 Wire Wire Line
@@
 Text GLabel 8125 1575 2    39   Input ~ 0
 VBUS
+$Comp
+L dk_TVS-Diodes:ESD5Z3_3T1G D?
+U 1 1 61F50F14
+P 1550 2325
+AR Path="/61C45066/61F50F14" Ref="D?"  Part="1"
+AR Path="/61F50F14" Ref="D?"  Part="1"
+AR Path="/61DDBD9F/61F50F14" Ref="D?"  Part="1"
+F 0 "D?" V 1603 2197 60  0000 R CNN
+F 1 "ESDA25P35" V 1497 2197 60  0000 R CNN
+F 2 "digikey-footprints:SOD-523" H 1750 2525 60  0001 L CNN
+F 3 "https://www.onsemi.com/pub/Collateral/ESD5Z2.5T1-D.PDF" H 1750 2625 60  0001 L CNN
+F 4 "ESD5Z3.3T1GOSCT-ND" H 1750 2725 60  0001 L CNN "Digi-Key_PN"
+F 5 "ESD5Z3.3T1G" H 1750 2825 60  0001 L CNN "MPN"
+F 6 "Circuit Protection" H 1750 2925 60  0001 L CNN "Category"
+F 7 "TVS - Diodes" H 1750 3025 60  0001 L CNN "Family"
+F 8 "https://www.onsemi.com/pub/Collateral/ESD5Z2.5T1-D.PDF" H 1750 3125 60  0001 L CNN "DK_Datasheet_Link"
+F 9 "/product-detail/en/on-semiconductor/ESD5Z3.3T1G/ESD5Z3.3T1GOSCT-ND/1967044" H 1750 3225 60  0001 L CNN "DK_Detail_Page"
+F 10 "TVS DIODE 3.3V 14.1V SOD523" H 1750 3325 60  0001 L CNN "Description"
+F 11 "ON Semiconductor" H 1750 3425 60  0001 L CNN "Manufacturer"
+F 12 "Active" H 1750 3525 60  0001 L CNN "Status"
+	1    1550 2325
+	0    -1   -1   0
+$EndComp
+Wire Wire Line
+	1550 2125 1550 1575
+Wire Wire Line
+	1375 1575 1550 1575
+Connection ~ 1550 1575
+Wire Wire Line
+	1550 1575 2375 1575
+$Comp
+L OLIMEX_Power:GND #PWR?
+U 1 1 61F58B30
+P 7150 3075
+AR Path="/619540C6/61F58B30" Ref="#PWR?"  Part="1"
+AR Path="/61F58B30" Ref="#PWR?"  Part="1"
+AR Path="/61DDBD9F/61F58B30" Ref="#PWR?"  Part="1"
+F 0 "#PWR?" H 7150 2825 50  0001 C CNN
+F 1 "GND" H 7155 2902 50  0000 C CNN
+F 2 "" H 7150 3075 60  0000 C CNN
+F 3 "" H 7150 3075 60  0000 C CNN
+	1    7150 3075
+	-1   0    0    -1
+$EndComp
+Wire Wire Line
+	1550 2525 1550 3050
+$Comp
+L OLIMEX_Power:GND #PWR?
+U 1 1 61F5A776
+P 1550 3050
+AR Path="/619540C6/61F5A776" Ref="#PWR?"  Part="1"
+AR Path="/61F5A776" Ref="#PWR?"  Part="1"
+AR Path="/61DDBD9F/61F5A776" Ref="#PWR?"  Part="1"
+F 0 "#PWR?" H 1550 2800 50  0001 C CNN
+F 1 "GND" H 1555 2877 50  0000 C CNN
+F 2 "" H 1550 3050 60  0000 C CNN
+F 3 "" H 1550 3050 60  0000 C CNN
+	1    1550 3050
+	-1   0    0    -1
+$EndComp
 $EndSCHEMATC

Commit message: ALL DONE BUT THE HDMI SECTION. NEED FOOTPRINT ASSIGNMENT
Parts:
- gave numbers to parts that had none: 16
Connections:
- net VBUS is gone; now on net SYS_PWR: D16.1 (K)
- net SYS_PWR: no longer C100.2, D15.K, D16.2 (A), Q9.7 (D), Q9.8 (D), R77.1
- new net PWR_FRM_SNK: C100.2, D15.K, D16.2 (A), Q9.7 (D), Q9.8 (D), R77.1
Other:
- note added: "THIS ENSURES THE THE VARIABLE POWER SUPPLY\nIS ONLY POWERED FROM THE SINK PD CNTRL\n(THE V_BUS FROM THE HOST CANNOT PWR THE\nVAR PWR BUCK SUPPLY)"
Changed lines of the file:
@@
 $Descr A4 11693 8268
 encoding utf-8
-Sheet 3 11
+Sheet 8 15
 Title ""
 Date ""
@@
 Comment4 ""
 $EndDescr
-Text GLabel 7150 1575 1    50   Input ~ 0
-SYS_PWR
 Wire Wire Line
 	2800 3075 3725 3075
@@
 P 2800 2275
 AR Path="/61DE3B32" Ref="R?"  Part="1"
-AR Path="/61DDBD9F/61DE3B32" Ref="R?"  Part="1"
-F 0 "R?" H 2868 2321 50  0000 L CNN
+AR Path="/61DDBD9F/61DE3B32" Ref="R72"  Part="1"
+F 0 "R72" H 2868 2321 50  0000 L CNN
 F 1 "470" H 2868 2230 50  0000 L CNN
 F 2 "" V 2840 2265 50  0001 C CNN
@@
 P 2375 2825
 AR Path="/61DE3B39" Ref="C?"  Part="1"
-AR Path="/61DDBD9F/61DE3B39" Ref="C?"  Part="1"
-F 0 "C?" H 2490 2871 50  0000 L CNN
+AR Path="/61DDBD9F/61DE3B39" Ref="C97"  Part="1"
+F 0 "C97" H 2490 2871 50  0000 L CNN
 F 1 "1uF" H 2490 2780 50  0000 L CNN
 F 2 "" H 2413 2675 50  0001 C CNN
@@
 P 2800 2800
 AR Path="/61DE3B3F" Ref="R?"  Part="1"
-AR Path="/61DDBD9F/61DE3B3F" Ref="R?"  Part="1"
-F 0 "R?" H 2868 2846 50  0000 L CNN
+AR Path="/61DDBD9F/61DE3B3F" Ref="R73"  Part="1"
+F 0 "R73" H 2868 2846 50  0000 L CNN
 F 1 "1K" H 2868 2755 50  0000 L CNN
 F 2 "" V 2840 2790 50  0001 C CNN
@@
 P 2375 2325
 AR Path="/61DE3B46" Ref="D?"  Part="1"
-AR Path="/61DDBD9F/61DE3B46" Ref="D?"  Part="1"
-F 0 "D?" V 2475 2300 50  0000 R CNN
+AR Path="/61DDBD9F/61DE3B46" Ref="D14"  Part="1"
+F 0 "D14" V 2475 2300 50  0000 R CNN
 F 1 "MBRAF440T3G" V 2225 2450 50  0000 R CNN
 F 2 "" H 2375 2325 50  0001 C CNN
@@
 P 4175 1850
 AR Path="/61DE3B5D" Ref="#PWR?"  Part="1"
-AR Path="/61DDBD9F/61DE3B5D" Ref="#PWR?"  Part="1"
-F 0 "#PWR?" H 4175 1700 50  0001 C CNN
+AR Path="/61DDBD9F/61DE3B5D" Ref="#PWR0194"  Part="1"
+F 0 "#PWR0194" H 4175 1700 50  0001 C CNN
 F 1 "+3.3V" H 4190 2023 50  0000 C CNN
 F 2 "" H 4175 1850 60  0000 C CNN
@@
 P 6075 1575
 AR Path="/61DE3B63" Ref="Q?"  Part="1"
-AR Path="/61DDBD9F/61DE3B63" Ref="Q?"  Part="1"
-F 0 "Q?" V 6317 1325 50  0000 C CNN
+AR Path="/61DDBD9F/61DE3B63" Ref="Q9"  Part="1"
+F 0 "Q9" V 6317 1325 50  0000 C CNN
 F 1 "STL6P3LLH6" V 6226 1325 50  0000 C CNN
 F 2 "" H 6075 1575 50  0001 C CNN
@@
 P 5300 1800
 AR Path="/61DE3B69" Ref="R?"  Part="1"
-AR Path="/61DDBD9F/61DE3B69" Ref="R?"  Part="1"
-F 0 "R?" H 5368 1846 50  0000 L CNN
+AR Path="/61DDBD9F/61DE3B69" Ref="R74"  Part="1"
+F 0 "R74" H 5368 1846 50  0000 L CNN
 F 1 "100K" H 5368 1755 50  0000 L CNN
 F 2 "" V 5340 1790 50  0001 C CNN
@@
 P 5300 2325
 AR Path="/61DE3B6F" Ref="R?"  Part="1"
-AR Path="/61DDBD9F/61DE3B6F" Ref="R?"  Part="1"
-F 0 "R?" H 5368 2371 50  0000 L CNN
+AR Path="/61DDBD9F/61DE3B6F" Ref="R75"  Part="1"
+F 0 "R75" H 5368 2371 50  0000 L CNN
 F 1 "22K" H 5368 2280 50  0000 L CNN
 F 2 "" V 5340 2315 50  0001 C CNN
@@
 P 6175 2050
 AR Path="/61DE3B7B" Ref="R?"  Part="1"
-AR Path="/61DDBD9F/61DE3B7B" Ref="R?"  Part="1"
-F 0 "R?" H 6243 2096 50  0000 L CNN
+AR Path="/61DDBD9F/61DE3B7B" Ref="R76"  Part="1"
+F 0 "R76" H 6243 2096 50  0000 L CNN
 F 1 "22K" H 6243 2005 50  0000 L CNN
 F 2 "" V 6215 2040 50  0001 C CNN
@@
 P 6550 2050
 AR Path="/61DE3B87" Ref="C?"  Part="1"
-AR Path="/61DDBD9F/61DE3B87" Ref="C?"  Part="1"
-F 0 "C?" V 6802 2050 50  0000 C CNN
+AR Path="/61DDBD9F/61DE3B87" Ref="C100"  Part="1"
+F 0 "C100" V 6802 2050 50  0000 C CNN
 F 1 "0.1uF" V 6711 2050 50  0000 C CNN
 F 2 "" H 6588 1900 50  0001 C CNN
@@
 AR Path="/619540C6/61DE3B8E" Ref="#PWR?"  Part="1"
 AR Path="/61DE3B8E" Ref="#PWR?"  Part="1"
-AR Path="/61DDBD9F/61DE3B8E" Ref="#PWR?"  Part="1"
-F 0 "#PWR?" H 4325 3675 50  0001 C CNN
+AR Path="/61DDBD9F/61DE3B8E" Ref="#PWR0195"  Part="1"
+F 0 "#PWR0195" H 4325 3675 50  0001 C CNN
 F 1 "GND" H 4330 3752 50  0000 C CNN
 F 2 "" H 4325 3925 60  0000 C CNN
@@
 AR Path="/619540C6/61DE3B95" Ref="#PWR?"  Part="1"
 AR Path="/61DE3B95" Ref="#PWR?"  Part="1"
-AR Path="/61DDBD9F/61DE3B95" Ref="#PWR?"  Part="1"
-F 0 "#PWR?" H 5125 1700 50  0001 C CNN
+AR Path="/61DDBD9F/61DE3B95" Ref="#PWR0196"  Part="1"
+F 0 "#PWR0196" H 5125 1700 50  0001 C CNN
 F 1 "GND" H 5130 1777 50  0000 C CNN
 F 2 "" H 5125 1950 60  0000 C CNN
@@
 P 4825 2000
 AR Path="/61DE3B9B" Ref="C?"  Part="1"
-AR Path="/61DDBD9F/61DE3B9B" Ref="C?"  Part="1"
-F 0 "C?" V 4775 2100 50  0000 C CNN
+AR Path="/61DDBD9F/61DE3B9B" Ref="C99"  Part="1"
+F 0 "C99" V 4775 2100 50  0000 C CNN
 F 1 "1uF" V 4875 2100 50  0000 C CNN
 F 2 "" H 4825 2000 50  0001 C CNN
@@
 P 6800 2325
 AR Path="/61DE3BA7" Ref="R?"  Part="1"
-AR Path="/61DDBD9F/61DE3BA7" Ref="R?"  Part="1"
-F 0 "R?" H 6868 2371 50  0000 L CNN
+AR Path="/61DDBD9F/61DE3BA7" Ref="R77"  Part="1"
+F 0 "R77" H 6868 2371 50  0000 L CNN
 F 1 "1K" H 6868 2280 50  0000 L CNN
 F 2 "" V 6840 2315 50  0001 C CNN
@@
 AR Path="/61C45066/61DE3BBC" Ref="D?"  Part="1"
 AR Path="/61DE3BBC" Ref="D?"  Part="1"
-AR Path="/61DDBD9F/61DE3BBC" Ref="D?"  Part="1"
-F 0 "D?" V 7203 2147 60  0000 R CNN
+AR Path="/61DDBD9F/61DE3BBC" Ref="D15"  Part="1"
+F 0 "D15" V 7203 2147 60  0000 R CNN
 F 1 "ESDA25P35" V 7097 2147 60  0000 R CNN
 F 2 "digikey-footprints:SOD-523" H 7350 2475 60  0001 L CNN
@@
 AR Path="/619540C6/61DE3BD5" Ref="#PWR?"  Part="1"
 AR Path="/61DE3BD5" Ref="#PWR?"  Part="1"
-AR Path="/61DDBD9F/61DE3BD5" Ref="#PWR?"  Part="1"
-F 0 "#PWR?" H 3500 3400 50  0001 C CNN
+AR Path="/61DDBD9F/61DE3BD5" Ref="#PWR0197"  Part="1"
+F 0 "#PWR0197" H 3500 3400 50  0001 C CNN
 F 1 "GND" H 3505 3477 50  0000 C CNN
 F 2 "" H 3500 3650 60  0000 C CNN
@@
 P 4475 1800
 AR Path="/61DE3BE2" Ref="C?"  Part="1"
-AR Path="/61DDBD9F/61DE3BE2" Ref="C?"  Part="1"
-F 0 "C?" H 4500 1900 50  0000 L CNN
+AR Path="/61DDBD9F/61DE3BE2" Ref="C98"  Part="1"
+F 0 "C98" H 4500 1900 50  0000 L CNN
 F 1 "1uF" H 4325 1900 50  0000 L CNN
 F 2 "" H 4513 1650 50  0001 C CNN
@@
 P 4325 2975
 AR Path="/61DE3BF7" Ref="U?"  Part="1"
-AR Path="/61DDBD9F/61DE3BF7" Ref="U?"  Part="1"
-F 0 "U?" H 4025 2100 50  0000 C CNN
+AR Path="/61DDBD9F/61DE3BF7" Ref="U12"  Part="1"
+F 0 "U12" H 4025 2100 50  0000 C CNN
 F 1 "STUSB4500QTR" H 3975 2025 50  0000 C CNN
 F 2 "Package_DFN_QFN:QFN-24-1EP_4x4mm_P0.5mm_EP2.7x2.7mm" H 4325 2975 50  0001 C CNN
@@
 Connection ~ 7150 1575
 $Comp
-L Device:D D?
+L Device:D D16
 U 1 1 61E1CE99
 P 7650 1575
-F 0 "D?" H 7650 1358 50  0000 C CNN
+F 0 "D16" H 7650 1358 50  0000 C CNN
 F 1 "SBR10B45P5-13" H 7650 1449 50  0000 C CNN
 F 2 "" H 7650 1575 50  0001 C CNN
@@
 	-1   0    0    1
 $EndComp
-Wire Wire Line
-	7800 1575 8125 1575
-Text GLabel 8125 1575 2    39   Input ~ 0
-VBUS
 $Comp
 L dk_TVS-Diodes:ESD5Z3_3T1G D?
@@
 AR Path="/61C45066/61F50F14" Ref="D?"  Part="1"
 AR Path="/61F50F14" Ref="D?"  Part="1"
-AR Path="/61DDBD9F/61F50F14" Ref="D?"  Part="1"
-F 0 "D?" V 1603 2197 60  0000 R CNN
+AR Path="/61DDBD9F/61F50F14" Ref="D13"  Part="1"
+F 0 "D13" V 1603 2197 60  0000 R CNN
 F 1 "ESDA25P35" V 1497 2197 60  0000 R CNN
 F 2 "digikey-footprints:SOD-523" H 1750 2525 60  0001 L CNN
@@
 AR Path="/619540C6/61F58B30" Ref="#PWR?"  Part="1"
 AR Path="/61F58B30" Ref="#PWR?"  Part="1"
-AR Path="/61DDBD9F/61F58B30" Ref="#PWR?"  Part="1"
-F 0 "#PWR?" H 7150 2825 50  0001 C CNN
+AR Path="/61DDBD9F/61F58B30" Ref="#PWR0198"  Part="1"
+F 0 "#PWR0198" H 7150 2825 50  0001 C CNN
 F 1 "GND" H 7155 2902 50  0000 C CNN
 F 2 "" H 7150 3075 60  0000 C CNN
@@
 AR Path="/619540C6/61F5A776" Ref="#PWR?"  Part="1"
 AR Path="/61F5A776" Ref="#PWR?"  Part="1"
-AR Path="/61DDBD9F/61F5A776" Ref="#PWR?"  Part="1"
-F 0 "#PWR?" H 1550 2800 50  0001 C CNN
+AR Path="/61DDBD9F/61F5A776" Ref="#PWR0199"  Part="1"
+F 0 "#PWR0199" H 1550 2800 50  0001 C CNN
 F 1 "GND" H 1555 2877 50  0000 C CNN
 F 2 "" H 1550 3050 60  0000 C CNN
@@
 	-1   0    0    -1
 $EndComp
+Text GLabel 8075 1575 2    50   Input ~ 0
+SYS_PWR
+Wire Wire Line
+	7800 1575 8075 1575
+Text GLabel 7150 1375 1    50   Input ~ 0
+PWR_FRM_SNK
+Wire Wire Line
+	7150 1575 7150 1375
+Text Notes 7225 975  0    39   ~ 0
+THIS ENSURES THE THE VARIABLE POWER SUPPLY\nIS ONLY POWERED FROM THE SINK PD CNTRL\n(THE V_BUS FROM THE HOST CANNOT PWR THE\nVAR PWR BUCK SUPPLY)
 $EndSCHEMATC
