File: SRC/USB_C_HUB/USB TO SATA.sch (KiCad schematic (older format))
At the start: 47 parts

Commit message: ALL DONE BUT THE HDMI SECTION. NEED FOOTPRINT ASSIGNMENT
Parts:
- gave numbers to parts that had none: 47

Commit message: schematic capture complete. Pending Footprint assignment. accetable Errors=21
Parts:
- added R101: 4.7K, symbol Device:R_US
- renumbered C149 to C100, C150 to C101, C151 to C102, C152 to C103, C153 to C104, C154 to C105, C155 to C106, C156 to C107, C157 to C108, C158 to C109, C159 to C110, C160 to C111, C161 to C112, C162 to C113, C163 to C114, C128 to C79, C129 to C80, C130 to C81, C131 to C82, C132 to C83, C133 to C84, C134 to C85, C135 to C86, C136 to C87, C137 to C88, C138 to C89, C139 to C90, C140 to C91, C141 to C92, C142 to C93, C143 to C94, C144 to C95, C145 to C96, C146 to C97, C147 to C98, C148 to C99, D21 to D23, R87 to R29, R88 to R30, R89 to R31, R90 to R32, R91 to R33, R92 to R34, R93 to R35, U14 to U9
Connections:
- net labels added: USS_SSRXM
- net labels removed: USS_SSSRXM
- wire segments 259 -> 262
- no-connect marks 50 -> 59
